Commit message: Launcher and urdf changes

File: src/city_simulation/models/autonomous_vehicle_old.urdf (robot description, URDF)
Before this commit: robot autonomous_vehicle, 7 links, 6 joints
Links:
- link chassisLink: mass 2 -> 2.0; geometry collision mesh filename=/home/alvaro/github/Programas-Modelado/Blender/Entrega/mesh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 scale=1.0 1.0 1.0; visual mesh filename=/home/alvaro/github/Programas-Modelado/Blender/Entrega/mesh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 scale=-0.01767 -0.01767 -0.01767
- link frontLeftWheelLink: geometry collision mesh filename=/home/alvaro/github/Programas-Modelado/Blender/Entrega/mesh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 scale=1.0 1.0 1.0; visual mesh filename=/home/alvaro/github/Programas-Modelado/Blender/Entrega/mesh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 scale=0.02333 0.02333 0.02333
- link frontRightWheelLink: geometry collision mesh filename=/home/alvaro/github/Programas-Modelado/Blender/Entrega/mesh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 scale=1.0 1.0 1.0; visual mesh filename=/home/alvaro/github/Programas-Modelado/Blender/Entrega/mesh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 scale=0.02333 0.02333 0.02333
- link rearLeftWheelLink: geometry collision mesh filename=/home/alvaro/github/Programas-Modelado/Blender/Entrega/mesh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 scale=1.0 1.0 1.0; visual mesh filename=/home/alvaro/github/Programas-Modelado/Blender/Entrega/mesh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 scale=0.02333 0.02333 0.02333
- link rearRightWheelLink: geometry collision mesh filename=/home/alvaro/github/Programas-Modelado/Blender/Entrega/mesh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 scale=1.0 1.0 1.0; visual mesh filename=/home/alvaro/github/Programas-Modelado/Blender/Entrega/mesh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 scale=0.02333 0.02333 0.02333
Joints:
- joint frontLeftWheelJoint: origin xyz=2.02598 -1.53082 -0.05739 rpy=1.5708 0 -1.5708 -> xyz=1.69167 -1.46869 -0.13224 rpy=-1.5708 0 -1.57121
- joint frontRightWheelJoint: origin xyz=-2.01372 -1.51765 -0.05739 rpy=1.5708 0 1.5708 -> xyz=-1.70064 -1.4471 -0.13224 rpy=-1.5708 0 1.57038
- joint onboardCameraJoint: origin xyz=0 -3.2 0.4 rpy=0 0 -1.57 -> xyz=0 -2.9 0.4 rpy=0 0 -1.57
- joint rearLeftWheelJoint: origin xyz=2.03577 0.86208 -0.05739 rpy=1.5708 0 -1.5708 -> xyz=1.73045 1.05373 -0.13224 rpy=-1.5708 0 -1.57121
- joint rearRightWheelJoint: origin xyz=-2.04563 0.93075 -0.05739 rpy=1.5708 0 1.5708 -> xyz=-1.69897 1.15481 -0.13224 rpy=-1.5708 0 1.57038

File: src/model/urdf/autonomous_vehicle.urdf (robot description, URDF)
Before this commit: robot autonomous_vehicle, 7 links, 6 joints
Links:
- link chassisLink: mass 6 -> 2
Joints:
- joint frontRightWheelJoint: origin xyz=-2.01372 -1.51765 -0.05451 rpy=1.5708 0 1.5708 -> xyz=-2.01372 -1.51765 -0.05739 rpy=1.5708 0 1.5708
- joint onboardCameraJoint: origin xyz=0 -2.9 0.4 rpy=0 0 -1.57 -> xyz=0 -3.2 0.4 rpy=0 0 -1.57
- joint rearLeftWheelJoint: origin xyz=2.03577 0.86208 -0.06106 rpy=1.5708 0 -1.5708 -> xyz=2.03577 0.86208 -0.05739 rpy=1.5708 0 -1.5708
- joint rearRightWheelJoint: origin xyz=-2.04563 0.93075 -0.04897 rpy=1.5708 0 1.5708 -> xyz=-2.04563 0.93075 -0.05739 rpy=1.5708 0 1.5708
