Commit message: Object Dataset and subfolder src

File: src/city_simulation/models/autonomous_vehicle.urdf (robot description, URDF)
Before this commit: robot autonomous_vehicle, 7 links, 6 joints
Links:
- link chassisLink: geometry collision mesh filename=model://autonomous_vehicle/meshes/dae/Bottom.003.dae scale=1.0 1.0 1.0; visual mesh filename=model://autonomous_vehicle/meshes/dae/Bottom.002.dae scale=0.01431 0.01431 0.01431
- link frontLeftWheelLink: geometry collision mesh filename=model://autonomous_vehicle/meshes/dae/chas-Cut.004.dae scale=1.0 1.0 1.0; visual mesh filename=model://autonomous_vehicle/meshes/dae/chas-Cut.003.dae scale=0.02678 0.02678 0.02678
- link frontRightWheelLink: geometry collision mesh filename=model://autonomous_vehicle/meshes/dae/chas-Cut.006.dae scale=1.0 1.0 1.0; visual mesh filename=model://autonomous_vehicle/meshes/dae/chas-Cut.dae scale=0.02678 0.02678 0.02678
- link rearLeftWheelLink: geometry collision mesh filename=model://autonomous_vehicle/meshes/dae/chas-Cut.005.dae scale=1.0 1.0 1.0; visual mesh filename=model://autonomous_vehicle/meshes/dae/chas-Cut.002.dae scale=0.02678 0.02678 0.02678
- link rearRightWheelLink: geometry collision mesh filename=model://autonomous_vehicle/meshes/dae/chas-Cut.007.dae scale=1.0 1.0 1.0; visual mesh filename=model://autonomous_vehicle/meshes/dae/chas-Cut.001.dae scale=0.02678 0.02678 0.02678
